Commit message: Get working ros2_control on real robot

File: description/gazebo_control.xacro (robot description, xacro)
@@ -6,5 +6,5 @@
             <left_joint>left_wheel_joint</left_joint>
             <right_joint>right_wheel_joint</right_joint>
-            <wheel_separation>0.075</wheel_separation>
+            <wheel_separation>0.17</wheel_separation>
             <wheel_diameter>0.065</wheel_diameter>
             <!-- Limits -->

File: description/lidar.xacro (robot description, xacro)
@@ -10,7 +10,5 @@
             <origin xyz="0.07 -0.24 -0.065" rpy="0 0 -${pi/2}"/>
             <geometry>
-                <!-- <cylinder radius="0.05" length="0.04"/> -->
-                <!-- <mesh filename="package://test_bot/stl/Rplidar.stl" scale="0.001 0.001 0.001" /> -->
-                <mesh filename="file://$(find test_bot)/stl/Rplidar.stl" scale="0.001 0.001 0.001" />
+                <mesh filename="file://$(find test_bot)/meshes/Rplidar.stl" scale="0.001 0.001 0.001" />
             </geometry>
             <material name="black"/>
@@ -19,6 +17,5 @@
             <geometry>
                 <!-- <cylinder radius="0.05" length="0.04"/> -->
-                <mesh filename="file://$(find test_bot)/stl/Rplidar.stl" scale="0.001 0.001 0.001" />
-                <!-- <mesh filename="package://find test_bot/stl/Rplidar.stl" scale="0.001 0.001 0.001" /> -->
+                <mesh filename="file://$(find test_bot)/meshes/Rplidar.stl" scale="0.001 0.001 0.001" />
             </geometry>
         </collision>
@@ -48,5 +45,5 @@
             <plugin name="laser_controller" filename="libgazebo_ros_ray_sensor.so">
                 <ros>
-                    <argument>--ros-args --remapping ~/out:=scan</argument>
+                    <remapping>~/out:=scan</remapping>
                 </ros>
                 <output_type>sensor_msgs/LaserScan</output_type>

File: description/robot_core.xacro (robot description, xacro)
@@ -39,7 +39,7 @@
     <link name="chassis">
         <visual>
-            <origin xyz="0.18 0.104 -0.005"/>
+            <origin xyz="0.08 0 0"/>
             <geometry>
-                <mesh filename="file://$(find test_bot)/stl/Chassis.stl" scale="0.001 0.001 0.001" />
+                <mesh filename="file://$(find test_bot)/meshes/Chassis.stl" scale="0.001 0.001 0.001" />
                 <!-- <mesh filename="$(find test_bot)/stl/Chassis.stl" scale="0.001 0.001 0.001" /> -->
             </geometry>
@@ -47,8 +47,7 @@
         </visual>
         <collision>
-            <origin xyz="0.18 0.104 -0.005"/>
+            <origin xyz="0.08 0 0"/>
             <geometry>
-                <!-- <mesh filename="$(find test_bot)/stl/Chassis.stl" scale="0.001 0.001 0.001" /> -->
-                <mesh filename="file://$(find test_bot)/stl/Chassis.stl" scale="0.001 0.001 0.001" />
+                <cylinder radius="0.08" length="0.003"/>
             </geometry>
         </collision>
@@ -58,12 +57,10 @@
             <inertia ixx="0.01" ixy="0" ixz="0" iyy="0.01" iyz="0" izz="0.01"/>
         </inertial> -->
-        <xacro:inertial_cylinder mass="0.3" length="0.005" radius="0.08">
-            <origin xyz="0.18 0 -0.005" rpy="0 0 0"/>
+        <xacro:inertial_cylinder mass="0.1" length="0.005" radius="0.08">
+            <origin xyz="0.08 0 0" rpy="0 0 0"/>
         </xacro:inertial_cylinder>
     </link>
     <gazebo reference="chassis">
         <material>Gazebo/Black</material>
-        <!-- <mu1>1.0</mu1>
-        <mu2>1.0</mu2> -->
     </gazebo>
     <!-- LEFT WHEEL LINK -->
@@ -71,5 +68,5 @@
         <parent link="base_link"/>
         <child link="left_wheel"/>
-        <origin xyz="0 0.045 0" rpy="-${pi/2} 0 0" />
+        <origin xyz="0 0.09 0" rpy="-${pi/2} 0 0" />
         <axis xyz="0 0 1"/>
     </joint>
@@ -77,5 +74,5 @@
         <visual>
             <geometry>
-                <cylinder radius="0.0325" length="0.025"/>
+                <cylinder radius="0.0325" length="0.02"/>
             </geometry>
             <material name="yellow"/>
@@ -86,5 +83,5 @@
             </geometry>
         </collision>
-        <xacro:inertial_cylinder mass="0.1" length="0.025" radius="0.0325">
+        <xacro:inertial_cylinder mass="0.1" length="0.02" radius="0.0325">
             <origin xyz="0 0 0" rpy="0 0 0"/>
         </xacro:inertial_cylinder>
@@ -97,5 +94,5 @@
         <parent link="base_link"/>
         <child link="right_wheel"/>
-        <origin xyz="0 -0.045 0" rpy="${pi/2} 0 0" />
+        <origin xyz="0 -0.09 0" rpy="${pi/2} 0 0" />
         <axis xyz="0 0 -1"/>
     </joint>
@@ -103,5 +100,5 @@
         <visual>
             <geometry>
-                <cylinder radius="0.0325" length="0.025"/>
+                <cylinder radius="0.0325" length="0.02"/>
             </geometry>
             <material name="yellow"/>
@@ -112,5 +109,5 @@
             </geometry>
         </collision>
-        <xacro:inertial_cylinder mass="0.1" length="0.025" radius="0.0325">
+        <xacro:inertial_cylinder mass="0.1" length="0.02" radius="0.0325">
             <origin xyz="0 0 0" rpy="0 0 0"/>
         </xacro:inertial_cylinder>

File: description/ros2_control.xacro (robot description, xacro)
@@ -1,5 +1,33 @@
 <?xml version="1.0"?>
 <robot xmlns:xacro="http://www.ros.org/wiki/xacro">
-    <ros2_control name="GazeboSystem" type="system">
+    <ros2_control name="RealRobot" type="system">
+        <hardware>
+            <plugin>diffdrive_arduino/DiffDriveArduinoHardware</plugin>
+            <param name="left_wheel_name">left_wheel_joint</param>
+            <param name="right_wheel_name">right_wheel_joint</param>
+            <param name="loop_rate">30</param>
+            <param name="device">/dev/serial/by-path/pci-0000:03:00.0-usb-0:2:1.0-port0</param>
+            <param name="baud_rate">57600</param>
+            <param name="timeout_ms">1000</param>
+            <param name="enc_counts_per_rev">3436</param>
+        </hardware>
+        <joint name="left_wheel_joint">
+            <command_interface name="velocity">
+                <param name="min">-10</param>
+                <param name="max">10</param>
+            </command_interface>
+            <state_interface name="position" />
+            <state_interface name="velocity" />
+        </joint>
+        <joint name="right_wheel_joint">
+            <command_interface name="velocity">
+                <param name="min">-10</param>
+                <param name="max">10</param>
+            </command_interface>
+            <state_interface name="position" />
+            <state_interface name="velocity" />
+        </joint>
+    </ros2_control>
+    <!-- <ros2_control name="GazeboSystem" type="system">
         <hardware>
             <plugin>gazebo_ros2_control/GazeboSystem</plugin>
@@ -21,5 +49,5 @@
             <state_interface name="position" />
         </joint>
-    </ros2_control>
+    </ros2_control> -->
     <gazebo>
         <plugin name="gazebo_ros2_control" filename="libgazebo_ros2_control.so">
