Commit message: Changes with rviz

File: description/lidar.xacro (robot description, xacro)
@@ -4,11 +4,11 @@
         <parent link="chassis"/>
         <child link="laser_frame"/>
-        <origin xyz="0.1 0 0.07" rpy="0 0 0"/>
+        <origin xyz="0.1 0 0.135" rpy="0 0 0"/>
     </joint>
     <link name="laser_frame">
         <visual>
-            <origin xyz="0.07 -0.24 -0.065" rpy="0 0 -${pi/2}"/>
             <geometry>
-                <mesh filename="file://$(find test_bot)/meshes/Rplidar.stl" scale="0.001 0.001 0.001" />
+                <mesh filename="package://test_bot/meshes/Rplidar.stl" scale="0.001 0.001 0.001" />
+                <!-- <mesh filename="file://$(find test_bot)/meshes/Rplidar.stl" scale="0.001 0.001 0.001" /> -->
             </geometry>
             <material name="black"/>
@@ -17,5 +17,6 @@
             <geometry>
                 <!-- <cylinder radius="0.05" length="0.04"/> -->
-                <mesh filename="file://$(find test_bot)/meshes/Rplidar.stl" scale="0.001 0.001 0.001" />
+                <mesh filename="package://test_bot/meshes/Rplidar.stl" scale="0.001 0.001 0.001" />
+                <!-- <mesh filename="file://$(find test_bot)/meshes/Rplidar.stl" scale="0.001 0.001 0.001" /> -->
             </geometry>
         </collision>

File: description/robot_core.xacro (robot description, xacro)
@@ -35,5 +35,5 @@
         <parent link="base_link"/>
         <child link="chassis"/>
-        <origin xyz="-0.08 0 0"/>
+        <origin xyz="-0.05 0 0"/>
     </joint>
     <link name="chassis">
@@ -41,5 +41,6 @@
             <origin xyz="0.08 0 0"/>
             <geometry>
-                <mesh filename="file://$(find test_bot)/meshes/Chassis.stl" scale="0.001 0.001 0.001" />
+                <mesh filename="package://test_bot/meshes/Chassis.stl" scale="0.001 0.001 0.001" />
+                <!-- <mesh filename="file://$(find test_bot)/meshes/Chassis.stl" scale="0.001 0.001 0.001" /> -->
                 <!-- <mesh filename="$(find test_bot)/stl/Chassis.stl" scale="0.001 0.001 0.001" /> -->
             </geometry>
@@ -76,5 +77,5 @@
                 <cylinder radius="0.0325" length="0.02"/>
             </geometry>
-            <material name="yellow"/>
+            <material name="blue"/>
         </visual>
         <collision>
@@ -88,5 +89,5 @@
     </link>
     <gazebo reference="left_wheel">
-        <material>Gazebo/Yellow</material>
+        <material>Gazebo/Blue</material>
     </gazebo>
     <!-- RIGHT WHEEL LINK -->
@@ -102,5 +103,5 @@
                 <cylinder radius="0.0325" length="0.02"/>
             </geometry>
-            <material name="yellow"/>
+            <material name="blue"/>
         </visual>
         <collision>
@@ -114,5 +115,5 @@
     </link>
     <gazebo reference="right_wheel">
-        <material>Gazebo/Yellow</material>
+        <material>Gazebo/Blue</material>
     </gazebo>
     <!-- CASTER WHEEL LINK -->
