Commit message: Some changes with hardware config

File: description/robot_core.xacro (robot description, xacro)
@@ -69,5 +69,5 @@
         <parent link="base_link"/>
         <child link="left_wheel"/>
-        <origin xyz="0 0.09 0" rpy="-${pi/2} 0 0" />
+        <origin xyz="0 0.1 0" rpy="-${pi/2} 0 0" />
         <axis xyz="0 0 1"/>
     </joint>
@@ -95,5 +95,5 @@
         <parent link="base_link"/>
         <child link="right_wheel"/>
-        <origin xyz="0 -0.09 0" rpy="${pi/2} 0 0" />
+        <origin xyz="0 -0.1 0" rpy="${pi/2} 0 0" />
         <axis xyz="0 0 -1"/>
     </joint>

File: description/ros2_control.xacro (robot description, xacro)
@@ -8,5 +8,5 @@
                 <param name="right_wheel_name">right_wheel_joint</param>
                 <param name="loop_rate">30</param>
-                <param name="device">/dev/serial/by-path/pci-0000:03:00.0-usb-0:2:1.0-port0</param>
+                <param name="device">/dev/serial/by-path/platform-fd500000.pcie-pci-0000:01:00.0-usb-0:1.2:1.0-port0</param>
                 <param name="baud_rate">57600</param>
                 <param name="timeout_ms">1000</param>

Commit message: Added joystick

File: description/robot_core.xacro (robot description, xacro)
@@ -43,5 +43,5 @@
                 <mesh filename="package://test_bot/meshes/Chassis.stl" scale="0.001 0.001 0.001" />
                 <!-- <mesh filename="file://$(find test_bot)/meshes/Chassis.stl" scale="0.001 0.001 0.001" /> -->
-                <!-- <mesh filename="$(find test_bot)/stl/Chassis.stl" scale="0.001 0.001 0.001" /> -->
+                <!-- <mesh filename="$(find test_bot)/meshes/Chassis.stl" scale="0.001 0.001 0.001" /> -->
             </geometry>
             <material name="black"/>
